File: 0022_Flame_Module_PT334.kicad_sch (KiCad schematic)
At the start: 13 parts, among them IC1 LM2903BHQDGKRQ1, Q1 Q_Photo_NPN, Q2 PDTC114EU,115

Commit message: Add files via upload
Parts:
- removed Q1: Q_Photo_NPN, symbol Device:Q_Photo_NPN
- added D2: LED, LED_SMD:LED_0805_2012Metric, symbol Device:LED
- added Q3: PT334-6B, meminle:PT3346B, symbol PT334-6B:PT334-6B
- added R4: 1k, Resistor_SMD:R_0805_2012Metric, symbol Device:R
- added U3: ~, Moduler_:pin_header, symbol moduler_pin:air
- C1, C2: footprint (none) -> Capacitor_SMD:C_0805_2012Metric
- D1: footprint (none) -> LED_SMD:LED_0805_2012Metric
- IC1: footprint SOP65P490X110-8N -> LM2903:SOP65P490X110-8N
- Q2: footprint PDTC114EU115 -> Package_TO_SOT_SMD:SOT-323_SC-70
- R1, R2, R3, R4, R5, R6: footprint (none) -> Resistor_SMD:R_0805_2012Metric
- RV1: footprint (none) -> meminle:3362P_1
Connections:
- net AN: now also U3.12
- net GND: now also D2.1 (K), U3.9
- net IN+: now also Q3.1 (E)
- net INT: now also U3.13
- net VCC renamed +5V
- net +5V: now also Q3.2 (C), R4.1, U3.7
- new net: D2.2 (A), R4.2
- no-connect marks 1 -> 15
Other:
- note added: "AIR PIN"
- note added: "SENSOR"
- moved on the sheet: C1, C2, D1, IC1, Q2, R1, R2, R3, R4, R5, R6, RV1
